Commit message: Fixed file not found for rviz

File: src/simple_arm/urdf/ur10.urdf (robot description, URDF)
Before this commit: robot ur10, 11 links, 10 joints
Links:
- link base_link: geometry collision mesh filename=file:///home/ubb/Documents/PersonalProject/install/simple_a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; visual mesh filename=file:///home/ubb/Documents/PersonalProject/install/simple_a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

File: src/simple_arm/urdf/ur10.urdf.xacro (robot description, xacro)
@@ -60,13 +60,13 @@
       <visual>
         <geometry>
-          <mesh filename="file://$(find simple_arm)/models/ur10/meshes/ur10/visual/base.dae" />
-        </geometry>
-        <material name="LightGrey">
-          <color rgba="0.7 0.7 0.7 1.0" />
-        </material>
-      </visual>
-      <collision>
-        <geometry>
-          <mesh filename="file://$(find simple_arm)/models/ur10/meshes/ur10/collision/base.stl" />
+          <mesh filename="file://$(find simple_arm)/models/ur10/meshes/visual/base.dae" />
+        </geometry>
+        <material name="LightGrey">
+          <color rgba="0.7 0.7 0.7 1.0" />
+        </material>
+      </visual>
+      <collision>
+        <geometry>
+          <mesh filename="file://$(find simple_arm)/models/ur10/meshes/collision/base.stl" />
         </geometry>
       </collision>
@@ -97,13 +97,13 @@
       <visual>
         <geometry>
-          <mesh filename="file://$(find simple_arm)/models/ur10/meshes/ur10/visual/shoulder.dae" />
-        </geometry>
-        <material name="LightGrey">
-          <color rgba="0.7 0.7 0.7 1.0" />
-        </material>
-      </visual>
-      <collision>
-        <geometry>
-          <mesh filename="file://$(find simple_arm)/models/ur10/meshes/ur10/collision/shoulder.stl" />
+          <mesh filename="file://$(find simple_arm)/models/ur10/meshes/visual/shoulder.dae" />
+        </geometry>
+        <material name="LightGrey">
+          <color rgba="0.7 0.7 0.7 1.0" />
+        </material>
+      </visual>
+      <collision>
+        <geometry>
+          <mesh filename="file://$(find simple_arm)/models/ur10/meshes/collision/shoulder.stl" />
         </geometry>
       </collision>
@@ -134,13 +134,13 @@
       <visual>
         <geometry>
-          <mesh filename="file://$(find simple_arm)/models/ur10/meshes/ur10/visual/upperarm.dae" />
-        </geometry>
-        <material name="LightGrey">
-          <color rgba="0.7 0.7 0.7 1.0" />
-        </material>
-      </visual>
-      <collision>
-        <geometry>
-          <mesh filename="file://$(find simple_arm)/models/ur10/meshes/ur10/collision/upperarm.stl" />
+          <mesh filename="file://$(find simple_arm)/models/ur10/meshes/visual/upperarm.dae" />
+        </geometry>
+        <material name="LightGrey">
+          <color rgba="0.7 0.7 0.7 1.0" />
+        </material>
+      </visual>
+      <collision>
+        <geometry>
+          <mesh filename="file://$(find simple_arm)/models/ur10/meshes/collision/upperarm.stl" />
         </geometry>
       </collision>
@@ -171,13 +171,13 @@
       <visual>
         <geometry>
-          <mesh filename="file://$(find simple_arm)/models/ur10/meshes/ur10/visual/forearm.dae" />
-        </geometry>
-        <material name="LightGrey">
-          <color rgba="0.7 0.7 0.7 1.0" />
-        </material>
-      </visual>
-      <collision>
-        <geometry>
-          <mesh filename="file://$(find simple_arm)/models/ur10/meshes/ur10/collision/forearm.stl" />
+          <mesh filename="file://$(find simple_arm)/models/ur10/meshes/visual/forearm.dae" />
+        </geometry>
+        <material name="LightGrey">
+          <color rgba="0.7 0.7 0.7 1.0" />
+        </material>
+      </visual>
+      <collision>
+        <geometry>
+          <mesh filename="file://$(find simple_arm)/models/ur10/meshes/collision/forearm.stl" />
         </geometry>
       </collision>
@@ -208,13 +208,13 @@
       <visual>
         <geometry>
-          <mesh filename="file://$(find simple_arm)/models/ur10/meshes/ur10/visual/wrist1.dae" />
-        </geometry>
-        <material name="LightGrey">
-          <color rgba="0.7 0.7 0.7 1.0" />
-        </material>
-      </visual>
-      <collision>
-        <geometry>
-          <mesh filename="file://$(find simple_arm)/models/ur10/meshes/ur10/collision/wrist1.stl" />
+          <mesh filename="file://$(find simple_arm)/models/ur10/meshes/visual/wrist1.dae" />
+        </geometry>
+        <material name="LightGrey">
+          <color rgba="0.7 0.7 0.7 1.0" />
+        </material>
+      </visual>
+      <collision>
+        <geometry>
+          <mesh filename="file://$(find simple_arm)/models/ur10/meshes/collision/wrist1.stl" />
         </geometry>
       </collision>
@@ -245,13 +245,13 @@
       <visual>
         <geometry>
-          <mesh filename="file://$(find simple_arm)/models/ur10/meshes/ur10/visual/wrist2.dae" />
-        </geometry>
-        <material name="LightGrey">
-          <color rgba="0.7 0.7 0.7 1.0" />
-        </material>
-      </visual>
-      <collision>
-        <geometry>
-          <mesh filename="file://$(find simple_arm)/models/ur10/meshes/ur10/collision/wrist2.stl" />
+          <mesh filename="file://$(find simple_arm)/models/ur10/meshes/visual/wrist2.dae" />
+        </geometry>
+        <material name="LightGrey">
+          <color rgba="0.7 0.7 0.7 1.0" />
+        </material>
+      </visual>
+      <collision>
+        <geometry>
+          <mesh filename="file://$(find simple_arm)/models/ur10/meshes/collision/wrist2.stl" />
         </geometry>
       </collision>
@@ -282,13 +282,13 @@
       <visual>
         <geometry>
-          <mesh filename="file://$(find simple_arm)/models/ur10/meshes/ur10/visual/wrist3.dae" />
-        </geometry>
-        <material name="LightGrey">
-          <color rgba="0.7 0.7 0.7 1.0" />
-        </material>
-      </visual>
-      <collision>
-        <geometry>
-          <mesh filename="file://$(find simple_arm)/models/ur10/meshes/ur10/collision/wrist3.stl" />
+          <mesh filename="file://$(find simple_arm)/models/ur10/meshes/visual/wrist3.dae" />
+        </geometry>
+        <material name="LightGrey">
+          <color rgba="0.7 0.7 0.7 1.0" />
+        </material>
+      </visual>
+      <collision>
+        <geometry>
+          <mesh filename="file://$(find simple_arm)/models/ur10/meshes/collision/wrist3.stl" />
         </geometry>
       </collision>
