Commit message: Robot spawning in gazebo

File: simple_arm/urdf/ur.transmission.xacro (robot description, xacro)
@@ -9,4 +9,5 @@
       <actuator name="${prefix}shoulder_pan_motor">
         <mechanicalReduction>1</mechanicalReduction>
+        <hardwareInterface>${hw_interface}</hardwareInterface>
       </actuator>
     </transmission>
@@ -17,4 +18,5 @@
       </joint>
       <actuator name="${prefix}shoulder_lift_motor">
+        <hardwareInterface>${hw_interface}</hardwareInterface>
         <mechanicalReduction>1</mechanicalReduction>
       </actuator>
@@ -26,4 +28,5 @@
       </joint>
       <actuator name="${prefix}elbow_motor">
+        <hardwareInterface>${hw_interface}</hardwareInterface>
         <mechanicalReduction>1</mechanicalReduction>
       </actuator>
@@ -35,4 +38,5 @@
       </joint>
       <actuator name="${prefix}wrist_1_motor">
+        <hardwareInterface>${hw_interface}</hardwareInterface>
         <mechanicalReduction>1</mechanicalReduction>
       </actuator>
@@ -44,4 +48,5 @@
       </joint>
       <actuator name="${prefix}wrist_2_motor">
+        <hardwareInterface>${hw_interface}</hardwareInterface>
         <mechanicalReduction>1</mechanicalReduction>
       </actuator>
@@ -53,4 +58,5 @@
       </joint>
       <actuator name="${prefix}wrist_3_motor">
+        <hardwareInterface>${hw_interface}</hardwareInterface>
         <mechanicalReduction>1</mechanicalReduction>
       </actuator>

File: simple_arm/urdf/ur10.urdf (robot description, URDF)
Before this commit: robot ur10, 11 links, 10 joints
Joints:
- joint shoulder_lift_joint: limit lower=-6.283185307179586 upper=6.283185307179586 effort=330.0 velocity=2.16 -> lower=-3.141592653589793 upper=3.141592653589793 effort=330.0 velocity=2.16
- joint shoulder_pan_joint: limit lower=-6.283185307179586 upper=6.283185307179586 effort=330.0 velocity=2.16 -> lower=-3.141592653589793 upper=3.141592653589793 effort=330.0 velocity=2.16
- joint wrist_1_joint: limit lower=-6.283185307179586 upper=6.283185307179586 effort=54.0 velocity=3.2 -> lower=-3.141592653589793 upper=3.141592653589793 effort=54.0 velocity=3.2
- joint wrist_2_joint: limit lower=-6.283185307179586 upper=6.283185307179586 effort=54.0 velocity=3.2 -> lower=-3.141592653589793 upper=3.141592653589793 effort=54.0 velocity=3.2
- joint wrist_3_joint: limit lower=-6.283185307179586 upper=6.283185307179586 effort=54.0 velocity=3.2 -> lower=-3.141592653589793 upper=3.141592653589793 effort=54.0 velocity=3.2

File: simple_arm/urdf/ur10_robot.urdf.xacro (robot description, xacro)
@@ -3,12 +3,18 @@
        name="ur10" >
   <xacro:arg name="transmission_hw_interface" default="hardware_interface/PositionJointInterface"/>
-  <!-- common stuff -->
-  <xacro:include filename="$(find simple_arm)/urdf/common.gazebo.xacro" />
   <!-- ur10 -->
   <xacro:include filename="$(find simple_arm)/urdf/ur10.urdf.xacro" />
   <!-- arm -->
-  <xacro:ur10_robot prefix="" joint_limited="false"
+  <xacro:ur10_robot prefix="" joint_limited="true"
     transmission_hw_interface="$(arg transmission_hw_interface)"
   />
+  <gazebo>
+    <plugin filename="libgazebo_ros2_control.so" name="gazebo_ros2_control">
+      <robot_sim_type>gazebo_ros2_control/DefaultRobotHWSim</robot_sim_type>
+      <robot_param>robot_description</robot_param>
+      <robot_param_node>robot_state_publisher</robot_param_node>
+      <parameters>$(find simple_arm)/configs/arm_controller_ur10.yaml</parameters>
+    </plugin>
+  </gazebo>
   <link name="world" />
   <joint name="world_joint" type="fixed">
