Commit message: Arm is moving

File: simple_arm/urdf/ur10.urdf (robot description, URDF)
Before this commit: robot ur10, 11 links, 10 joints
Joints:
- joint shoulder_lift_joint: limit lower=-3.141592653589793 upper=3.141592653589793 effort=330.0 velocity=2.16 -> lower=-6.283185307179586 upper=6.283185307179586 effort=330.0 velocity=2.16
- joint shoulder_pan_joint: limit lower=-3.141592653589793 upper=3.141592653589793 effort=330.0 velocity=2.16 -> lower=-6.283185307179586 upper=6.283185307179586 effort=330.0 velocity=2.16
- joint wrist_1_joint: limit lower=-3.141592653589793 upper=3.141592653589793 effort=54.0 velocity=3.2 -> lower=-6.283185307179586 upper=6.283185307179586 effort=54.0 velocity=3.2
- joint wrist_2_joint: limit lower=-3.141592653589793 upper=3.141592653589793 effort=54.0 velocity=3.2 -> lower=-6.283185307179586 upper=6.283185307179586 effort=54.0 velocity=3.2
- joint wrist_3_joint: limit lower=-3.141592653589793 upper=3.141592653589793 effort=54.0 velocity=3.2 -> lower=-6.283185307179586 upper=6.283185307179586 effort=54.0 velocity=3.2

File: simple_arm/urdf/ur10_robot.urdf.xacro (robot description, xacro)
@@ -6,10 +6,10 @@
   <xacro:include filename="$(find simple_arm)/urdf/ur10.urdf.xacro" />
   <!-- arm -->
-  <xacro:ur10_robot prefix="" joint_limited="true"
+  <xacro:ur10_robot prefix="" joint_limited="false"
     transmission_hw_interface="$(arg transmission_hw_interface)"
   />
   <gazebo>
     <plugin filename="libgazebo_ros2_control.so" name="gazebo_ros2_control">
-      <robot_sim_type>gazebo_ros2_control/DefaultRobotHWSim</robot_sim_type>
+      <!-- <robot_sim_type>gazebo_ros2_control/DefaultRobotHWSim</robot_sim_type> -->
       <robot_param>robot_description</robot_param>
       <robot_param_node>robot_state_publisher</robot_param_node>
