Commit message: Ur10 MoveIt sorta working

File: ur_configs/urdf/ur10.urdf.xacro (robot description, xacro)
@@ -1,6 +1,6 @@
 <?xml version="1.0"?>
 <robot xmlns:xacro="http://www.ros.org/wiki/xacro" name="RHEX">
-  <xacro:include filename="$(find simple_arm)/urdf/ur.transmission.xacro" />
-  <xacro:include filename="$(find simple_arm)/urdf/ur.gazebo.xacro" />
+  <xacro:include filename="$(find ur_configs)/urdf/ur.transmission.xacro" />
+  <xacro:include filename="$(find ur_configs)/urdf/ur.gazebo.xacro" />
   <xacro:macro name="cylinder_inertial" params="radius length mass *origin">
     <inertial>
@@ -60,13 +60,13 @@
       <visual>
         <geometry>
-          <mesh filename="file://$(find simple_arm)/models/ur10/meshes/visual/base.dae" />
-        </geometry>
-        <material name="LightGrey">
-          <color rgba="0.7 0.7 0.7 1.0" />
-        </material>
-      </visual>
-      <collision>
-        <geometry>
-          <mesh filename="file://$(find simple_arm)/models/ur10/meshes/collision/base.stl" />
+          <mesh filename="file://$(find ur_configs)/meshes/ur10/meshes/visual/base.dae" />
+        </geometry>
+        <material name="LightGrey">
+          <color rgba="0.7 0.7 0.7 1.0" />
+        </material>
+      </visual>
+      <collision>
+        <geometry>
+          <mesh filename="file://$(find ur_configs)/meshes/ur10/meshes/collision/base.stl" />
         </geometry>
       </collision>
@@ -97,13 +97,13 @@
       <visual>
         <geometry>
-          <mesh filename="file://$(find simple_arm)/models/ur10/meshes/visual/shoulder.dae" />
-        </geometry>
-        <material name="LightGrey">
-          <color rgba="0.7 0.7 0.7 1.0" />
-        </material>
-      </visual>
-      <collision>
-        <geometry>
-          <mesh filename="file://$(find simple_arm)/models/ur10/meshes/collision/shoulder.stl" />
+          <mesh filename="file://$(find ur_configs)/meshes/ur10/meshes/visual/shoulder.dae" />
+        </geometry>
+        <material name="LightGrey">
+          <color rgba="0.7 0.7 0.7 1.0" />
+        </material>
+      </visual>
+      <collision>
+        <geometry>
+          <mesh filename="file://$(find ur_configs)/meshes/ur10/meshes/collision/shoulder.stl" />
         </geometry>
       </collision>
@@ -134,13 +134,13 @@
       <visual>
         <geometry>
-          <mesh filename="file://$(find simple_arm)/models/ur10/meshes/visual/upperarm.dae" />
-        </geometry>
-        <material name="LightGrey">
-          <color rgba="0.7 0.7 0.7 1.0" />
-        </material>
-      </visual>
-      <collision>
-        <geometry>
-          <mesh filename="file://$(find simple_arm)/models/ur10/meshes/collision/upperarm.stl" />
+          <mesh filename="file://$(find ur_configs)/meshes/ur10/meshes/visual/upperarm.dae" />
+        </geometry>
+        <material name="LightGrey">
+          <color rgba="0.7 0.7 0.7 1.0" />
+        </material>
+      </visual>
+      <collision>
+        <geometry>
+          <mesh filename="file://$(find ur_configs)/meshes/ur10/meshes/collision/upperarm.stl" />
         </geometry>
       </collision>
@@ -171,13 +171,13 @@
       <visual>
         <geometry>
-          <mesh filename="file://$(find simple_arm)/models/ur10/meshes/visual/forearm.dae" />
-        </geometry>
-        <material name="LightGrey">
-          <color rgba="0.7 0.7 0.7 1.0" />
-        </material>
-      </visual>
-      <collision>
-        <geometry>
-          <mesh filename="file://$(find simple_arm)/models/ur10/meshes/collision/forearm.stl" />
+          <mesh filename="file://$(find ur_configs)/meshes/ur10/meshes/visual/forearm.dae" />
+        </geometry>
+        <material name="LightGrey">
+          <color rgba="0.7 0.7 0.7 1.0" />
+        </material>
+      </visual>
+      <collision>
+        <geometry>
+          <mesh filename="file://$(find ur_configs)/meshes/ur10/meshes/collision/forearm.stl" />
         </geometry>
       </collision>
@@ -208,13 +208,13 @@
       <visual>
         <geometry>
-          <mesh filename="file://$(find simple_arm)/models/ur10/meshes/visual/wrist1.dae" />
-        </geometry>
-        <material name="LightGrey">
-          <color rgba="0.7 0.7 0.7 1.0" />
-        </material>
-      </visual>
-      <collision>
-        <geometry>
-          <mesh filename="file://$(find simple_arm)/models/ur10/meshes/collision/wrist1.stl" />
+          <mesh filename="file://$(find ur_configs)/meshes/ur10/meshes/visual/wrist1.dae" />
+        </geometry>
+        <material name="LightGrey">
+          <color rgba="0.7 0.7 0.7 1.0" />
+        </material>
+      </visual>
+      <collision>
+        <geometry>
+          <mesh filename="file://$(find ur_configs)/meshes/ur10/meshes/collision/wrist1.stl" />
         </geometry>
       </collision>
@@ -245,13 +245,13 @@
       <visual>
         <geometry>
-          <mesh filename="file://$(find simple_arm)/models/ur10/meshes/visual/wrist2.dae" />
-        </geometry>
-        <material name="LightGrey">
-          <color rgba="0.7 0.7 0.7 1.0" />
-        </material>
-      </visual>
-      <collision>
-        <geometry>
-          <mesh filename="file://$(find simple_arm)/models/ur10/meshes/collision/wrist2.stl" />
+          <mesh filename="file://$(find ur_configs)/meshes/ur10/meshes/visual/wrist2.dae" />
+        </geometry>
+        <material name="LightGrey">
+          <color rgba="0.7 0.7 0.7 1.0" />
+        </material>
+      </visual>
+      <collision>
+        <geometry>
+          <mesh filename="file://$(find ur_configs)/meshes/ur10/meshes/collision/wrist2.stl" />
         </geometry>
       </collision>
@@ -282,13 +282,13 @@
       <visual>
         <geometry>
-          <mesh filename="file://$(find simple_arm)/models/ur10/meshes/visual/wrist3.dae" />
-        </geometry>
-        <material name="LightGrey">
-          <color rgba="0.7 0.7 0.7 1.0" />
-        </material>
-      </visual>
-      <collision>
-        <geometry>
-          <mesh filename="file://$(find simple_arm)/models/ur10/meshes/collision/wrist3.stl" />
+          <mesh filename="file://$(find ur_configs)/meshes/ur10/meshes/visual/wrist3.dae" />
+        </geometry>
+        <material name="LightGrey">
+          <color rgba="0.7 0.7 0.7 1.0" />
+        </material>
+      </visual>
+      <collision>
+        <geometry>
+          <mesh filename="file://$(find ur_configs)/meshes/ur10/meshes/collision/wrist3.stl" />
         </geometry>
       </collision>

File: ur_configs/urdf/ur10_robot.urdf.xacro (robot description, xacro)
@@ -4,15 +4,15 @@
   <xacro:arg name="transmission_hw_interface" default="hardware_interface/PositionJointInterface"/>
   <!-- ur10 -->
-  <xacro:include filename="$(find simple_arm)/urdf/ur10.urdf.xacro" />
+  <xacro:include filename="$(find ur_configs)/urdf/ur10.urdf.xacro" />
   <!-- arm -->
   <xacro:ur10_robot prefix="" joint_limited="true"
     transmission_hw_interface="$(arg transmission_hw_interface)"
   />
-  <gazebo>
+  <!-- <gazebo>
     <plugin filename="libgazebo_ros2_control.so" name="gazebo_ros2_control">
       <robot_sim_type>gazebo_ros2_control/DefaultRobotHWSim</robot_sim_type>
       <robot_param>robot_description</robot_param>
       <robot_param_node>robot_state_publisher</robot_param_node>
-      <parameters>$(find simple_arm)/configs/arm_controller_ur10.yaml</parameters>
+      <parameters>$(find ur_configs)/configs/arm_controller_ur10.yaml</parameters>
     </plugin>
   </gazebo>
@@ -22,4 +22,4 @@
     <child link = "base_link" />
     <origin xyz="0.0 0.0 0.0" rpy="0.0 0.0 0.0" />
-  </joint>
+  </joint> -->
 </robot>
