Commit message: Added a new package for moveit with UR10WIP not working

File: ur_configs/urdf/ur10.urdf (robot description, URDF)
Before this commit: robot ur10, 10 links, 9 joints
Links:
- removed link base
- added link world
Joints:
- removed joint base_link-base_fixed_joint
- added joint world_joint: type fixed, parent world, child base_link, origin xyz=0.0 0.0 0.0 rpy=0.0 0.0 0.0
