Commit message: Webots trajectory control working

File: ur_configs/urdf/panda/panda_arm_hand.urdf (robot description, URDF)
Before this commit: robot panda, 12 links, 12 joints
Links:
- added link world

File: ur_configs/urdf/panda/panda_arm_hand.urdf.xacro (robot description, xacro)
@@ -5,7 +5,16 @@
   <xacro:include filename="$(find ur_configs)/urdf/panda/panda.gazebo.xacro"/>
   <xacro:include filename="$(find ur_configs)/urdf/panda/panda.control.xacro"/>
+  <link name="world"/>
   <xacro:panda_arm xyz="0 0 0" rpy="0 0 0" connected_to="world" arm_id="panda"/>
   <xacro:hand ns="panda" rpy="0 0 ${-pi/4}" connected_to="panda_link8"/>
   <xacro:panda_gazebo arm_id="panda"/>
   <xacro:panda_control arm_id="panda"/>
+  <gazebo>
+    <plugin filename="libgazebo_ros2_control.so" name="gazebo_ros2_control">
+      <robot_sim_type>gazebo_ros2_control/DefaultRobotHWSim</robot_sim_type>
+      <robot_param>robot_description</robot_param>
+      <robot_param_node>robot_state_publisher</robot_param_node>
+      <parameters>$(find ur_configs)/configs/arm_controller_panda.yaml</parameters>
+    </plugin>
+  </gazebo>
 </robot>
