Commit message: Fixed panda model not finding files

File: ur_configs/urdf/panda/hand.xacro (robot description, xacro)
@@ -12,10 +12,10 @@
       <visual>
         <geometry>
-          <mesh filename="package://ur_configs/meshes/panda/meshes/visual/hand.dae"/>
+          <mesh filename="file://$(find ur_configs)/meshes/panda/meshes/visual/hand.dae"/>
         </geometry>
       </visual>
       <collision>
         <geometry>
-          <mesh filename="package://ur_configs/meshes/panda/meshes/collision/hand.stl"/>
+          <mesh filename="file://$(find ur_configs)/meshes/panda/meshes/collision/hand.stl"/>
         </geometry>
       </collision>
@@ -29,10 +29,10 @@
       <visual>
         <geometry>
-          <mesh filename="package://ur_configs/meshes/panda/meshes/visual/finger.dae"/>
+          <mesh filename="file://$(find ur_configs)/meshes/panda/meshes/visual/finger.dae"/>
         </geometry>
       </visual>
       <collision>
         <geometry>
-          <mesh filename="package://ur_configs/meshes/panda/meshes/collision/finger.stl"/>
+          <mesh filename="file://$(find ur_configs)/meshes/panda/meshes/collision/finger.stl"/>
         </geometry>
       </collision>
@@ -47,5 +47,5 @@
         <origin xyz="0 0 0" rpy="0 0 ${pi}"/>
         <geometry>
-          <mesh filename="package://ur_configs/meshes/panda/meshes/visual/finger.dae"/>
+          <mesh filename="file://$(find ur_configs)/meshes/panda/meshes/visual/finger.dae"/>
         </geometry>
       </visual>
@@ -53,5 +53,5 @@
         <origin xyz="0 0 0" rpy="0 0 ${pi}"/>
         <geometry>
-          <mesh filename="package://ur_configs/meshes/panda/meshes/collision/finger.stl"/>
+          <mesh filename="file://$(find ur_configs)/meshes/panda/meshes/collision/finger.stl"/>
         </geometry>
       </collision>

File: ur_configs/urdf/panda/panda_arm_hand.urdf (robot description, URDF)
Before this commit: robot panda, 13 links, 12 joints
Links:
- link panda_hand: geometry collision mesh filename=file:///home/ubb/Documents/PersonalProject/install/ur_confi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; visual mesh filename=file:///home/ubb/Documents/PersonalProject/install/ur_confi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
- link panda_leftfinger: geometry collision mesh filename=file:///home/ubb/Documents/PersonalProject/install/ur_confi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; visual mesh filename=file:///home/ubb/Documents/PersonalProject/install/ur_confi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
- link panda_rightfinger: geometry collision mesh filename=file:///home/ubb/Documents/PersonalProject/install/ur_confi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; visual mesh filename=file:///home/ubb/Documents/PersonalProject/install/ur_confi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

Commit message: Updating for gazebo

File: ur_configs/urdf/panda/hand.xacro (robot description, xacro)
@@ -75,5 +75,4 @@
       <axis xyz="0 -1 0"/>
       <limit effort="20" lower="0.0" upper="0.04" velocity="0.2"/>
-      <mimic joint="${ns}_finger_joint1" />
     </joint>
   </xacro:macro>

File: ur_configs/urdf/panda/panda_arm_hand.urdf (robot description, URDF)
Before this commit: robot panda, 13 links, 12 joints
Joints:
- joint panda_finger_joint2: mimic joint=panda_finger_joint1 -> (none)
