Commit message: Fixed tf tree and removed useless messages

File: ur_configs/urdf/panda/panda.urdf (robot description, URDF)
Before this commit: robot panda, 12 links, 11 joints
Links:
- added link base_link
- added link world
Joints:
- added joint panda_to_world: type fixed, parent base_link, child world, origin xyz=0 0 0 rpy=0 0 0
- added joint world_to_base: type fixed, parent world, child panda_link0, origin xyz=0 0 0 rpy=0 0 0

Commit message: Fixed throw in webots

File: ur_configs/urdf/panda/panda.urdf (robot description, URDF)
Before this commit: robot panda, 14 links, 13 joints
Links:
- removed link base_link
- removed link world
Joints:
- removed joint panda_to_world
- removed joint world_to_base
